File: power_supply_project/power_supply.kicad_pcb (KiCad board)
At the start: 2 copper layers, 110 x 45 mm, 12 parts, among them J1 Screw_Terminal_01x02, J2 Screw_Terminal_01x02, J4 Conn_01x01_Pin, J5 Conn_01x01_Pin, J6 Conn_01x01_Pin, J7 Conn_01x01_Pin, T1 Transformer_1P_1S, U1 MB10S-13

Commit message: update pcb layout to include linear regulator
Parts:
- added G***: LOGO, kicad_libraries:farm_hacks, F.Cu at (162.4, 56.6)
- added J3: Conn_01x01_Pin, Connector_PinHeader_2.54mm:PinHeader_1x01_P2.54mm_Vertical, F.Cu at (186.8, 90.3)
- added J8: Conn_01x01_Pin, Connector_PinHeader_2.54mm:PinHeader_1x01_P2.54mm_Vertical, F.Cu at (189.3, 63.8)
- added J9: Conn_01x02_Pin, Connector_PinHeader_2.54mm:PinHeader_1x02_P2.54mm_Vertical, F.Cu at (169.3, 89.1)
- added R2: 2k, Resistor_THT:R_Axial_DIN0207_L6.3mm_D2.5mm_P7.62mm_Horizontal, F.Cu at (185.0, 73.8)
- added R4: 2.2k, Resistor_THT:R_Axial_DIN0207_L6.3mm_D2.5mm_P7.62mm_Horizontal, F.Cu at (180.0, 71.2)
- added R5: CT-6EP103, kody_custom:POT_CT-6EP103_NDC, F.Cu at (180.0, 87.5)
- added U2: LM317_TO-220, Package_TO_SOT_THT:TO-220-3_Vertical, F.Cu at (180.1, 65.0)
- moved J1 16.4 mm to (194.4, 76.2)
Connections:
- net Net-(J1-Pin_2) renamed GND
- net Net-(J2-Pin_1) renamed AC_2
- net Net-(T1-AA) renamed AC_3
- J1 pad 1: Net-(D1-A) -> Power_output
Routing:
- net GND: track 49.9 -> 0.00 mm, vias 0 -> 6
- net AC_3: track 15.0 -> 27.1 mm
- net Net-(U2-ADJ): track 0.00 -> 11.6 mm
- net Net-(J9-Pin_1): track 0.00 -> 9.90 mm
- net Net-(R4-Pad2): track 0.00 -> 3.69 mm
- net Net-(D1-A): track 42.8 -> 40.7 mm
- added copper zone on F.Cu, net AC_2
- added copper zone on F.Cu, net AC_3
- added copper zone on B.Cu, net GND
- added copper zone on F.Cu, net GND
- added copper zone on F.Cu, net Power_output
- added copper zone on F.Cu, net VAC
Other:
- board size 110 x 45 mm -> 127.5 x 45 mm
- board text added: "+ DC after Regulator"
- board text added: "- DC after Regulator"
- board text added: "PPK2 Port Current from Voltage Adjustment"
- board text added: "Power Supply Project Revision 1 Designed by Kody Rogers"

Commit message: added notes and such
Changed lines of the file:
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@@
 		(tags "Through hole pin header THT 1x01 2.54mm single row")
 		(property "Reference" "J6"
-			(at 0 -2.33 0)
+			(at -2.89 -0.01 0)
 			(layer "F.SilkS")
 			(effects
@@
 	)
 	(gr_text "Power Supply Project Revision 1\nDesigned by Kody Rogers"
-		(at 169.722502 54.853373 0)
+		(at 169.175 54.575 0)
 		(layer "F.SilkS")
 		(effects
@@
 	)
 	(gr_text "Positive DC"
-		(at 151.62 61.35 0)
+		(at 150.95 62.475 0)
 		(layer "F.SilkS")
 		(effects
