File: dusk_to_dawn/op_amp_version/op_amp_version.kicad_sch (KiCad schematic)
At the start: 12 parts, among them J1 Conn_01x02_Pin, J2 Conn_01x02_Pin, J3 Conn_01x02_Pin, J4 Conn_01x02_Pin, U2 TLC372CP

Commit message: add first version of op amp dusk to dawn
Parts:
- added C1: 0.01u, Capacitor_SMD:C_0805_2012Metric_Pad1.18x1.45mm_HandSolder, symbol Device:C
- BT1: footprint Battery:Battery_Panasonic_CR2032-HFN_Horizontal_CircularHoles -> Connector_Wire:SolderWire-0.1sqmm_1x02_P3.6mm_D0.4mm_OD1mm
- R2: value 33k -> 330k
- R3: value 22k -> 33k
- R4: value 22k -> 330k
Connections:
- net 3V: now also J2.1 (Pin_1), J3.2 (Pin_2), J4.1 (Pin_1), C1.1; no longer R1.1, R3.1
- net GND: now also C1.2; no longer D1.1 (K)
- net at J3.1 (Pin_1): now also R1.1; no longer U2.3 (+)
- net at R1.2, R2.1: now also U2.3 (+); no longer J3.2 (Pin_2)
- net at R5.1: now also D1.2 (A); no longer J2.1 (Pin_1)
- net at J2.2 (Pin_2): now also R5.2; no longer U2.1
- net at R3.2, R4.1: now also U2.2 (-); no longer J4.1 (Pin_1)
- net at J4.2 (Pin_2): now also R3.1; no longer U2.2 (-)
- new net: D1.1 (K), U2.1
Other:
- note added: "1.7V"
- note removed: "1.8V"
- moved on the sheet: D1, J2, J3, J4, R5
